File: Hardware/Servo_Trigger.sch (EAGLE design)
At the start: 21 parts, among them U1 ATTINY84, Y1 16MHZ

Commit message: Revision from collaborator and checklists
Added mounting holes, rearranged the interface connectors.
Parts:
- added JP4: M021X02_NO_SILK, SparkFun-Connectors:M021X02_NO_SILK
- added STANDOFF1, STANDOFF2, STANDOFF3, STANDOFF4: STAND-OFF, SparkFun-Electromechanical:STAND-OFF
- R4, R5, R6: value 10k -> 10K; device SparkFun-Resistors:10KOHM1/10W1%(0603)0603 -> SparkFun-Resistors:10KOHM-1/10W-1%(0603)0603
Connections:
- net GND: now also JP4.1
- net VCC: now also JP4.2
Other:
- note added: "Expecting 5VDC power. Current consumed is dependent on servo type and loading."
- note added: "Power Input/ Daisy-Chain Output"
- note added: "V10"
- note removed: "Power Input"
- note removed: "V01"
- moved on the sheet: JP3
Changed lines of the file:
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@@
 <?xml version="1.0" encoding="utf-8"?>
 <!DOCTYPE eagle SYSTEM "eagle.dtd">
-<eagle version="6.5.0">
+<eagle version="7.1.0">
 <drawing>
 <settings>
@@
 <layer number="56" name="wert" color="7" fill="1" visible="no" active="no"/>
 <layer number="57" name="tCAD" color="7" fill="1" visible="no" active="no"/>
+<layer number="90" name="Modules" color="5" fill="1" visible="yes" active="yes"/>
 <layer number="91" name="Nets" color="2" fill="1" visible="yes" active="yes"/>
 <layer number="92" name="Busses" color="1" fill="1" visible="yes" active="yes"/>
@@
 <parts>
 <part name="FRAME1" library="SparkFun-Aesthetics" deviceset="FRAME-LETTER" device=""/>
-<part name="R4" library="SparkFun-Resistors" deviceset="10KOHM1/10W1%(0603)" device="0603" value="10k"/>
+<part name="R4" library="SparkFun-Resistors" deviceset="10KOHM-1/10W-1%(0603)" device="0603" value="10K"/>
 <part name="JP9" library="SparkFun-Connectors" deviceset="AVR_SPI_PRG_6" device="PTH" value=""/>
 <part name="U1" library="SparkFun-DigitalIC" deviceset="ATTINY84" device=""/>
@@
 <part name="FID1" library="SparkFun-Aesthetics" deviceset="FIDUCIAL" device="UFIDUCIAL"/>
 <part name="FID2" library="SparkFun-Aesthetics" deviceset="FIDUCIAL" device="UFIDUCIAL"/>
-<part name="R5" library="SparkFun-Resistors" deviceset="10KOHM1/10W1%(0603)" device="0603" value="10k"/>
+<part name="R5" library="SparkFun-Resistors" deviceset="10KOHM-1/10W-1%(0603)" device="0603" value="10K"/>
 <part name="SUPPLY11" library="SparkFun-Aesthetics" deviceset="VCC" device=""/>
-<part name="R6" library="SparkFun-Resistors" deviceset="10KOHM1/10W1%(0603)" device="0603" value="10k"/>
+<part name="R6" library="SparkFun-Resistors" deviceset="10KOHM-1/10W-1%(0603)" device="0603" value="10K"/>
 <part name="SUPPLY12" library="SparkFun-Aesthetics" deviceset="VCC" device=""/>
 <part name="SJ1" library="SparkFun-Passives" deviceset="JUMPER-PAD-2-NO" device="YES_SILK" value="N.O."/>
@@
 <part name="C1" library="SparkFun-Capacitors" deviceset="10UF-16V-10%(TANT)" device="" value="10uF"/>
 <part name="Y1" library="SparkFun-FreqCtrl" deviceset="RESONATOR" device="16MHZ" value="16MHZ"/>
+<part name="STANDOFF1" library="SparkFun-Electromechanical" deviceset="STAND-OFF" device=""/>
+<part name="STANDOFF2" library="SparkFun-Electromechanical" deviceset="STAND-OFF" device=""/>
+<part name="STANDOFF3" library="SparkFun-Electromechanical" deviceset="STAND-OFF" device=""/>
+<part name="STANDOFF4" library="SparkFun-Electromechanical" deviceset="STAND-OFF" device=""/>
+<part name="JP4" library="SparkFun-Connectors" deviceset="M02" device="1X02_NO_SILK" value="M021X02_NO_SILK"/>
+<part name="SUPPLY13" library="SparkFun-Aesthetics" deviceset="VCC" device=""/>
+<part name="GND9" library="SparkFun-Aesthetics" deviceset="GND" device=""/>
 </parts>
 <sheets>
@@
 <plain>
 <text x="165.1" y="7.62" size="2.54" layer="94" font="vector">Byron Jacquot</text>
-<text x="238.76" y="7.62" size="2.54" layer="94" font="vector">V01</text>
-<text x="7.62" y="177.8" size="2.54" layer="94" font="vector">Power Input</text>
+<text x="238.76" y="7.62" size="2.54" layer="94" font="vector">V10</text>
+<text x="7.62" y="177.8" size="2.54" layer="94" font="vector">Power Input/
+Daisy-Chain Output</text>
 <text x="63.5" y="175.26" size="2.54" layer="94" font="vector">ISP Connection</text>
 <text x="157.48" y="127" size="2.54" layer="94" font="vector">Control Potentiometers</text>
@@
 <text x="124.46" y="139.7" size="1.27" layer="94">Pulled up internally in processor
 Datasheet says Rup is in the 20K to 50K range.</text>
+<text x="5.08" y="139.7" size="1.27" layer="94">Expecting 5VDC power.
+Current consumed is dependent
+on servo type and loading.</text>
 </plain>
 <instances>
@@
 <instance part="GND5" gate="1" x="210.82" y="147.32"/>
 <instance part="SUPPLY9" gate="G$1" x="210.82" y="165.1"/>
-<instance part="JP3" gate="G$1" x="22.86" y="157.48"/>
-<instance part="SUPPLY10" gate="G$1" x="33.02" y="165.1"/>
-<instance part="GND6" gate="1" x="33.02" y="152.4"/>
+<instance part="JP3" gate="G$1" x="7.62" y="157.48" smashed="yes">
+<attribute name="NAME" x="5.08" y="163.322" size="1.778" layer="95"/>
+</instance>
+<instance part="SUPPLY10" gate="G$1" x="17.78" y="165.1"/>
+<instance part="GND6" gate="1" x="17.78" y="152.4"/>
 <instance part="LOGO1" gate="G$1" x="160.02" y="45.72"/>
 <instance part="LOGO2" gate="G$1" x="190.5" y="35.56"/>
@@
 <instance part="C1" gate="G$1" x="129.54" y="93.98"/>
 <instance part="Y1" gate="G$1" x="20.32" y="83.82"/>
+<instance part="STANDOFF1" gate="G$1" x="243.84" y="25.4"/>
+<instance part="STANDOFF2" gate="G$1" x="246.38" y="25.4"/>
+<instance part="STANDOFF3" gate="G$1" x="246.38" y="27.94"/>
+<instance part="STANDOFF4" gate="G$1" x="243.84" y="27.94"/>
+<instance part="JP4" gate="G$1" x="43.18" y="157.48" smashed="yes" rot="MR0">
+<attribute name="NAME" x="45.72" y="163.322" size="1.778" layer="95" rot="MR0"/>
+</instance>
+<instance part="SUPPLY13" gate="G$1" x="33.02" y="165.1"/>
+<instance part="GND9" gate="1" x="33.02" y="152.4"/>
 </instances>
 <busses>
@@
 <pinref part="JP3" gate="G$1" pin="2"/>
 <pinref part="SUPPLY10" gate="G$1" pin="VCC"/>
-<wire x1="30.48" y1="160.02" x2="33.02" y2="160.02" width="0.1524" layer="91"/>
-<wire x1="33.02" y1="160.02" x2="33.02" y2="165.1" width="0.1524" layer="91"/>
+<wire x1="15.24" y1="160.02" x2="17.78" y2="160.02" width="0.1524" layer="91"/>
+<wire x1="17.78" y1="160.02" x2="17.78" y2="165.1" width="0.1524" layer="91"/>
 </segment>
 <segment>
@@
 <pinref part="SUPPLY6" gate="G$1" pin="VCC"/>
 <wire x1="185.42" y1="99.06" x2="185.42" y2="109.22" width="0.1524" layer="91"/>
+</segment>
+<segment>
+<pinref part="JP4" gate="G$1" pin="2"/>
+<pinref part="SUPPLY13" gate="G$1" pin="VCC"/>
+<wire x1="35.56" y1="160.02" x2="33.02" y2="160.02" width="0.1524" layer="91"/>
+<wire x1="33.02" y1="160.02" x2="33.02" y2="165.1" width="0.1524" layer="91"/>
 </segment>
 </net>
@@
 <pinref part="JP3" gate="G$1" pin="1"/>
 <pinref part="GND6" gate="1" pin="GND"/>
-<wire x1="30.48" y1="157.48" x2="33.02" y2="157.48" width="0.1524" layer="91"/>
-<wire x1="33.02" y1="157.48" x2="33.02" y2="154.94" width="0.1524" layer="91"/>
+<wire x1="15.24" y1="157.48" x2="17.78" y2="157.48" width="0.1524" layer="91"/>
+<wire x1="17.78" y1="157.48" x2="17.78" y2="154.94" width="0.1524" layer="91"/>
 </segment>
 <segment>
@@
 <wire x1="185.42" y1="81.28" x2="185.42" y2="88.9" width="0.1524" layer="91"/>
 </segment>
+<segment>
+<pinref part="JP4" gate="G$1" pin="1"/>
+<pinref part="GND9" gate="1" pin="GND"/>
+<wire x1="35.56" y1="157.48" x2="33.02" y2="157.48" width="0.1524" layer="91"/>
+<wire x1="33.02" y1="157.48" x2="33.02" y2="154.94" width="0.1524" layer="91"/>
+</segment>
 </net>
