File: Hardware/SparkFun_Servo_Trigger.sch (EAGLE design)
At the start: 30 parts, among them U1 ATTINY84, Y1 16MHZ

Commit message: Replacing Designer name and version number.
They were part of the Frame, but it lost it's attributes in the library
update.
Other:
- note added: "Byron Jacquot"
- note added: "V11"
Changed lines of the file:
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@@
 "T" sets the time it takes to move from A to B
  and back, over a range of 0 to 10 seconds.</text>
+<text x="167.64" y="7.62" size="3.81" layer="94" font="vector">Byron Jacquot</text>
+<text x="238.76" y="7.62" size="2.54" layer="94" font="vector">V11</text>
 </plain>
 <instances>
